File: kicad/vwcdpic/tht/emulator.kicad_pcb (KiCad board)
At the start: 2 copper layers, 49.8 x 49.8 mm, 44 parts, among them P1 digi, P2 Ain, P3 Aout, U1 PIC12F629, U2 78L05, U3 TL072, U4 TL071

Commit message: no idea ...
Parts:
- moved U2 26.1 mm to (158.6, 85.5)
- moved R6 19.4 mm to (165.9, 95.0)
- moved C4 19.2 mm to (146.3, 86.1)
- moved C3 19.2 mm to (152.7, 85.3)
- moved R1 19.2 mm to (146.6, 96.8)
- moved R7 19.2 mm to (165.9, 98.3)
- moved C2 19.1 mm to (170.4, 85.6)
- moved P1 19.1 mm to (173.5, 90.7)
- moved C1 19.0 mm to (164.6, 85.6)
- moved R5 19.0 mm to (165.9, 91.4)
- moved U1 18.9 mm to (154.2, 94.5)
- moved R9 15.8 mm to (128.8, 122.9)
- moved C9 9.97 mm to (164.7, 148.3), turned to 270 degrees
- moved R2 7.39 mm to (156.2, 141.4), turned to 0 degrees
- moved R17 4.38 mm to (146.3, 108.2), turned to 180 degrees
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Connections:
- U2 pad 1: (no net) -> POWER_CTL
- U2 pad 2: (no net) -> GND
- U2 pad 3: (no net) -> +5V
Routing:
- net filtered_12V: track 120.3 -> 134.6 mm
- net +5V: track 42.7 -> 31.2 mm
- net Net-(C14-Pad2): track 19.0 -> 8.62 mm
- net Net-(C11-Pad1): track 19.1 -> 10.9 mm
- net Net-(C10-Pad1): track 26.8 -> 21.9 mm
- net POWER_CTL: track 21.5 -> 16.8 mm
- net Net-(C14-Pad1): track 35.1 -> 30.4 mm
- net Net-(R15-Pad2): track 14.7 -> 11.9 mm
- net +12V: track 24.4 -> 27.2 mm
- net CLK: track 8.20 -> 5.62 mm
- net DataIn: track 4.99 -> 3.28 mm
- net Net-(R14-Pad1): track 12.3 -> 13.9 mm
- net Net-(C7-Pad2): track 26.6 -> 27.3 mm
- net Net-(C12-Pad1): track 14.2 -> 13.6 mm
- net Net-(C8-Pad1): track 12.5 -> 13.1 mm
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- added copper zone on F.Cu, net GND
Other:
- board size 49.8 x 49.8 mm -> 52.1 x 73.7 mm

Commit message: ..
Parts:
- P1: footprint Connect:SIL-7 -> Pin_Headers:Pin_Header_Straight_1x07
- U2: footprint Discret:TO92-123 -> my_modules:TO92-STABIL
- moved U2 2.95 mm to (155.7, 85.4), turned to 225 degrees
Routing:
- net +5V: track 31.2 -> 28.2 mm
- net POWER_CTL: track 16.8 -> 19.7 mm
Other:
- board size 52.1 x 73.7 mm -> 52.3 x 73.7 mm
