File: kicad/vwcdpic/separated_audio_board/separated_audio_board.sch (KiCad schematic (older format))
At the start: 33 parts, among them P1 CONN_6, P2 IN, P3 OUT, P4 POWER, U1 PIC12F629, U2 78L05, U3 TL072

Commit message: update
Parts:
- removed P1: CONN_6, symbol CONN_6
- removed P2: IN, symbol CONN_3
- removed P3: OUT, symbol CONN_3
- removed P4: POWER, symbol CONN_2
- added P1: CONN_01X05, symbol CONN_01X05
- added P2, P3: CONN_01X03, symbol CONN_01X03
- added P4: CONN_01X02, symbol CONN_01X02
