File: kicad/bt_breakout_adapter_xs3868/bt_breakout_adapter_xs3868.kicad_pcb (KiCad board)
At the start: 2 copper layers, 26.9 x 36.3 mm, 4 parts, among them P1 CONN_01X12, P2 CONN_01X12, U1 XS3860

Commit message: pj3020b jack
Parts:
- J1: footprint my_modules:3.5mm_stereo_jack_PJ242 -> jacks:3.5mm_stereo_jack_PJ3020B
- moved J1 0.92 mm to (156.2, 102.9)
Routing:
- net Net-(J1-Pad5): track 34.3 -> 29.1 mm
- net Net-(J1-Pad2): track 44.3 -> 49.4 mm
- net Net-(J1-Pad1): track 51.1 -> 46.9 mm
