File: kicad/motorola_cracker/motorola_cracker_as_arduino_shield/motorola_cracker_as_arduino_shield.sch (KiCad schematic (older format))
At the start: 16 parts, among them P1 CONN_01X01, P2 CONN_2, SW1 SWITCH_INV, SW2 SWITCH_INV, U1 78L10, U5 68HC05_PLCC, X1 4Mhz

Commit message: motorola cracker simple board for usb to serial dongle (tested with cp2102)
Parts:
- C1, C2, C3, C4: symbol C -> C-RESCUE-motorola_cracker_as_arduino_shield
- R2, R7, R8, R9: symbol R -> R-RESCUE-motorola_cracker_as_arduino_shield
Changed lines of the file:
@@
 EESchema Schematic File Version 2
+LIBS:motorola_cracker_as_arduino_shield-rescue
 LIBS:power
 LIBS:device
@@
 LIBS:memory
 LIBS:xilinx
-LIBS:special
 LIBS:microcontrollers
 LIBS:dsp
@@
 $EndComp
 $Comp
-L C C4
+L C-RESCUE-motorola_cracker_as_arduino_shield C4
 U 1 1 52DC255A
 P 2650 7200
@@
 $EndComp
 $Comp
-L C C3
+L C-RESCUE-motorola_cracker_as_arduino_shield C3
 U 1 1 52DC2436
 P 6350 4150
@@
 $EndComp
 $Comp
-L C C2
+L C-RESCUE-motorola_cracker_as_arduino_shield C2
 U 1 1 52DC2429
 P 6350 3550
@@
 $EndComp
 $Comp
-L R R7
+L R-RESCUE-motorola_cracker_as_arduino_shield R7
 U 1 1 52DAF9A3
 P 6750 3150
@@
 $EndComp
 $Comp
-L R R8
+L R-RESCUE-motorola_cracker_as_arduino_shield R8
 U 1 1 52DAF95D
 P 7000 1700
@@
 $EndComp
 $Comp
-L R R9
+L R-RESCUE-motorola_cracker_as_arduino_shield R9
 U 1 1 52DAF927
 P 9550 4350
@@
 $EndComp
 $Comp
-L R R2
+L R-RESCUE-motorola_cracker_as_arduino_shield R2
 U 1 1 52DAF78A
 P 6750 4850
@@
 $EndComp
 $Comp
-L C C1
+L C-RESCUE-motorola_cracker_as_arduino_shield C1
 U 1 1 52DAF214
 P 1500 7200
