File: kicad/VWCDChangerRaspberryPi/VWCDChangerRaspberryPi.sch (KiCad schematic (older format))
At the start: 42 parts, among them IC1 ATMEGA328P-A, P1 CONN_02X20, P2 CONN_02X40, U1 LD1117S33TR, U2 CAT24C32, Y1 16Mhz

Commit message: deleted obsolete files
Parts:
- removed Q? (x3): BSS138, SOT-23, symbol BSS138
- removed R? (x6): 3k9, Resistors_SMD:R_1206_HandSoldering, symbol R
- added C10: 1uF/6.3V, Capacitors_Tantalum_SMD:TantalC_SizeA_EIA-3216_Reflow, symbol CP
- added C?: 100n, Capacitors_SMD:C_1206, symbol C
- added D?: TL431DBZ, SOT-23, symbol TL431DBZ
- added L?: INDUCTOR, Inductors_NEOSID:Neosid_Inductor_SM-NE30_SMD1210, symbol INDUCTOR
- added P?: CONN_01X05, symbol CONN_01X05
- added P? (x3): CONN_01X06, symbol CONN_01X06
- added P?: CONN_01X03, symbol CONN_01X03
- added Q? (x20): BSS138, SOT-23, symbol BSS138
- added R? (x3): 3k3, Resistors_SMD:R_0201, symbol R
- added R? (x18): 0, Resistors_SMD:R_0201, symbol R
- added R? (x40): 3k9, Resistors_SMD:R_1206, symbol R
- added R?: 1k8, Resistors_SMD:R_1206, symbol R
- C1, C4: footprint (none) -> Capacitors_Tantalum_SMD:TantalC_SizeD_EIA-7343_Reflow
- C2, C3, C5, C7: footprint 1206 -> Capacitors_SMD:C_1206
- C6: footprint 1206 -> Capacitors_SMD:C_0805
- C8: renamed from C?; footprint (none) -> Capacitors_SMD:C_1206
- C9: renamed from C?; footprint 1206 -> Capacitors_SMD:C_1206
- D1, D2: renamed from D?; footprint (none) -> Diodes_SMD:DO-214AB
- JP1: footprint (none) -> Resistors_SMD:R_0201
- JP2: footprint (none) -> Socket_Strips:Socket_Strip_Straight_1x02
- R1, R2, R3, R4: footprint Resistors_SMD:R_1206_HandSoldering -> Resistors_SMD:R_1206
- R13, R14, R15, R7, R8, R9: renamed from R?; footprint Resistors_SMD:R_1206_HandSoldering -> Resistors_SMD:R_1206
- gave numbers to parts that had none: 4
Connections:
- net labels added: ARDUINO_VCC, AREF, AVCC, FIS_CLK, FIS_DATA, FIS_ENABLE, INT0, INT1, SPI_MISO, SPI_MOSI, SPI_SCK
- net labels removed: MISO, PD2, PD3
- wire segments 197 -> 386
Other:
- moved on the sheet: C1, C2, C3, C4, C5, C6, C7, C8, C9, CON1, D1, D2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
