File: kicad/vwcdpic/pic_emulator_smd_no_audio/emulator.sch (KiCad schematic (older format))
At the start: 10 parts, among them P1 CONN_01X05, P2 CONN_01X04, U1 PIC12F629, U2 LM78L05ACZ

Commit message: merge v2 and v3 to single board
Parts:
- added C1: 1uF/6.3V, Capacitors_Tantalum_SMD:TantalC_SizeA_EIA-3216_Reflow, symbol CP
- added R5_v2, R6_v2: 3k3, Resistors_SMD:R_0805, symbol R-RESCUE-emulator
- added UART_v2: CONN_01X04, Pin_Headers:Pin_Header_Straight_1x02, symbol CONN_01X02
- C10, C2: footprint Capacitors_SMD:C_1206_HandSoldering -> Capacitors_SMD:C_0805
- R1, R7: footprint Resistors_SMD:R_1206_HandSoldering -> Resistors_SMD:R_0805
- R5_v3: renamed from R5; footprint Resistors_SMD:R_1206_HandSoldering -> Resistors_SMD:R_0805
- R6_v3: renamed from R6; footprint Resistors_SMD:R_1206_HandSoldering -> Resistors_SMD:R_0805
- U2: footprint SMD_Packages:SOT-223 -> my_modules:SOT-223-REGULATOR; symbol LM78L05ACZ -> 78L05
- renumbered P2 to ICSP_UART_v3, P1 to RADIO1
Connections:
- wire segments 32 -> 45
Changed lines of the file:
@@
 F 0 "C10" H 4150 2600 50  0000 L CNN
 F 1 "100n" H 4150 2400 50  0000 L CNN
-F 2 "Capacitors_SMD:C_1206_HandSoldering" H 4100 2500 60  0001 C CNN
+F 2 "Capacitors_SMD:C_0805" H 4100 2500 60  0001 C CNN
 F 3 "" H 4100 2500 60  0001 C CNN
 	1    4100 2500
@@
 Text GLabel 7650 3600 0    60   Input ~ 0
 DataOut
-Text GLabel 5650 3950 2    60   Input ~ 0
+Text GLabel 5750 3950 2    60   Input ~ 0
 DataOut
-Text GLabel 5650 3250 2    60   Input ~ 0
+Text GLabel 5750 3250 2    60   Input ~ 0
 CLK
-Text GLabel 5650 3650 2    60   Input ~ 0
+Text GLabel 5750 3650 2    60   Input ~ 0
 DataIn
 $Comp
@@
 F 0 "C2" H 5100 5650 50  0000 L CNN
 F 1 "100n" H 5100 5450 50  0000 L CNN
-F 2 "Capacitors_SMD:C_1206_HandSoldering" H 5050 5550 60  0001 C CNN
+F 2 "Capacitors_SMD:C_0805" H 5050 5550 60  0001 C CNN
 F 3 "" H 5050 5550 60  0001 C CNN
 	1    5050 5550
@@
 F 0 "R7" V 5380 3950 50  0000 C CNN
 F 1 "3k3" V 5300 3950 50  0000 C CNN
-F 2 "Resistors_SMD:R_1206_HandSoldering" H 5300 3950 60  0001 C CNN
+F 2 "Resistors_SMD:R_0805" H 5300 3950 60  0001 C CNN
 F 3 "" H 5300 3950 60  0001 C CNN
 	1    5300 3950
@@
 $EndComp
 $Comp
-L R-RESCUE-emulator R5
+L R-RESCUE-emulator R5_v3
 U 1 1 52D02AC2
 P 5300 3250
-F 0 "R5" V 5380 3250 50  0000 C CNN
+F 0 "R5_v3" V 5380 3250 50  0000 C CNN
 F 1 "3k3" V 5300 3250 50  0000 C CNN
-F 2 "Resistors_SMD:R_1206_HandSoldering" H 5300 3250 60  0001 C CNN
+F 2 "Resistors_SMD:R_0805" H 5300 3250 60  0001 C CNN
 F 3 "" H 5300 3250 60  0001 C CNN
 	1    5300 3250
@@
 $EndComp
 $Comp
-L R-RESCUE-emulator R6
+L R-RESCUE-emulator R6_v3
 U 1 1 52D02ABB
 P 5300 3650
-F 0 "R6" V 5380 3650 50  0000 C CNN
+F 0 "R6_v3" V 5380 3650 50  0000 C CNN
 F 1 "3k3" V 5300 3650 50  0000 C CNN
-F 2 "Resistors_SMD:R_1206_HandSoldering" H 5300 3650 60  0001 C CNN
+F 2 "Resistors_SMD:R_0805" H 5300 3650 60  0001 C CNN
 F 3 "" H 5300 3650 60  0001 C CNN
 	1    5300 3650
@@
 $EndComp
 $Comp
-L CONN_01X05 P1
+L CONN_01X05 RADIO1
 U 1 1 542D55A4
 P 7900 3600
-F 0 "P1" H 7900 3900 50  0000 C CNN
+F 0 "RADIO1" H 7900 3900 50  0000 C CNN
 F 1 "CONN_01X05" V 8000 3600 50  0000 C CNN
 F 2 "Pin_Headers:Pin_Header_Straight_1x05" H 7900 3600 60  0001 C CNN
@@
 F 0 "R1" V 3230 3000 50  0000 C CNN
 F 1 "10k" V 3150 3000 50  0000 C CNN
-F 2 "Resistors_SMD:R_1206_HandSoldering" H 3150 3000 60  0001 C CNN
+F 2 "Resistors_SMD:R_0805" H 3150 3000 60  0001 C CNN
 F 3 "" H 3150 3000 60  0001 C CNN
 	1    3150 3000
@@
 $EndComp
 $Comp
-L CONN_01X04 P2
+L CONN_01X04 ICSP_UART_v3
 U 1 1 542D83A2
 P 2650 3600
-F 0 "P2" H 2650 3900 50  0000 C CNN
+F 0 "ICSP_UART_v3" H 2650 3900 50  0000 C CNN
 F 1 "CONN_01X04" V 2750 3600 50  0000 C CNN
 F 2 "Pin_Headers:Pin_Header_Straight_1x04" H 2650 3600 60  0001 C CNN
@@
 $EndComp
 $Comp
-L LM78L05ACZ U2
+L 78L05 U2
 U 1 1 546C9D74
 P 5500 5200
 F 0 "U2" H 5300 5400 40  0000 C CNN
 F 1 "LM78L05ACZ" H 5500 5400 40  0000 L CNN
-F 2 "SMD_Packages:SOT-223" H 5500 5300 30  0000 C CIN
+F 2 "my_modules:SOT-223-REGULATOR" H 5500 5300 30  0000 C CIN
 F 3 "" H 5500 5200 60  0000 C CNN
 	1    5500 5200
@@
 	7650 3800 7700 3800
 Wire Wire Line
-	5650 3950 5550 3950
-Wire Wire Line
-	5650 3650 5550 3650
+	5550 3950 5750 3950
+Wire Wire Line
+	5550 3650 5750 3650
 Wire Wire Line
 	5050 5750 5050 5950
@@
 	4850 3950 5050 3950
 Wire Wire Line
-	5650 3250 5550 3250
+	5550 3250 5750 3250
 Wire Wire Line
 	7650 3700 7700 3700
@@
 	3150 2750 3150 2500
 Wire Wire Line
-	3150 3250 3150 3950
+	3150 3250 3150 4000
 Wire Wire Line
 	3400 3250 3400 3450
@@
 Wire Wire Line
 	2950 3750 2850 3750
+$Comp
+L CP C1
+U 1 1 55C4B796
+P 3150 4150
+F 0 "C1" H 3175 4250 50  0000 L CNN
+F 1 "1uF/6.3V" H 3175 4050 50  0000 L CNN
+F 2 "Capacitors_Tantalum_SMD:TantalC_SizeA_EIA-3216_Reflow" H 3188 4000 30  0000 C CNN
+F 3 "" H 3150 4150 60  0000 C CNN
+	1    3150 4150
+	1    0    0    -1
+$EndComp
+$Comp
+L GND #PWR07
+U 1 1 55C4B8F3
+P 3150 4400
+F 0 "#PWR07" H 3150 4400 30  0001 C CNN
+F 1 "GND" H 3150 4330 30  0001 C CNN
+F 2 "" H 3150 4400 60  0001 C CNN
+F 3 "" H 3150 4400 60  0001 C CNN
+	1    3150 4400
+	1    0    0    -1
+$EndComp
+Wire Wire Line
+	3150 4400 3150 4300
+Connection ~ 3150 3950
+$Comp
+L R-RESCUE-emulator R5_v2
+U 1 1 55C4BA7B
+P 5300 4400
+F 0 "R5_v2" V 5380 4400 50  0000 C CNN
+F 1 "3k3" V 5300 4400 50  0000 C CNN
+F 2 "Resistors_SMD:R_0805" H 5300 4400 60  0001 C CNN
+F 3 "" H 5300 4400 60  0001 C CNN
+	1    5300 4400
+	0    -1   -1   0
+$EndComp
+$Comp
+L R-RESCUE-emulator R6_v2
+U 1 1 55C4BADB
+P 5300 4700
+F 0 "R6_v2" V 5380 4700 50  0000 C CNN
+F 1 "3k3" V 5300 4700 50  0000 C CNN
+F 2 "Resistors_SMD:R_0805" H 5300 4700 60  0001 C CNN
+F 3 "" H 5300 4700 60  0001 C CNN
+	1    5300 4700
+	0    -1   -1   0
+$EndComp
+Wire Wire Line
+	5550 4400 5600 4400
+Wire Wire Line
+	5600 4400 5600 3250
+Connection ~ 5600 3250
+Wire Wire Line
+	5550 4700 5650 4700
+Wire Wire Line
+	5650 4700 5650 3650
+Connection ~ 5650 3650
+Wire Wire Line
+	2900 4400 5050 4400
+Wire Wire Line
+	5050 4700 3000 4700
+Wire Wire Line
+	3000 4700 3000 3550
+Connection ~ 3000 3550
+Wire Wire Line
+	2900 3450 2900 4400
+Connection ~ 2900 3450
+$Comp
+L CONN_01X02 UART_v2
+U 1 1 55C4D672
+P 5350 2800
+F 0 "UART_v2" H 5350 3100 50  0000 C CNN
+F 1 "CONN_01X04" V 5450 2800 50  0000 C CNN
+F 2 "Pin_Headers:Pin_Header_Straight_1x02" H 5350 2800 60  0001 C CNN
+F 3 "" H 5350 2800 60  0000 C CNN
+	1    5350 2800
+	1    0    0    -1
+$EndComp
+Wire Wire Line
+	5150 2750 4950 2750
+Wire Wire Line
+	4950 2750 4950 3250
+Connection ~ 4950 3250
+Wire Wire Line
+	5000 3650 5000 2850
+Wire Wire Line
+	5000 2850 5150 2850
+Connection ~ 5000 3650
 $EndSCHEMATC

Commit message: revert to version 3 based
Parts:
- removed R5_v2, R6_v2: 3k3, Resistors_SMD:R_0805, symbol R-RESCUE-emulator
- removed UART_v2: CONN_01X04, Pin_Headers:Pin_Header_Straight_1x02, symbol CONN_01X02
- renumbered ICSP_UART_v3 to ICSP_UART1, R5_v3 to R5, R6_v3 to R6
Connections:
- net MCLR_VPP: no longer names the net of C1.1, ICSP_UART1.2 (P2), R1.1, U1.4 (GP3/MCLR)
Changed lines of the file:
@@
 $EndComp
 $Comp
-L R-RESCUE-emulator R5_v3
+L R-RESCUE-emulator R5
 U 1 1 52D02AC2
 P 5300 3250
-F 0 "R5_v3" V 5380 3250 50  0000 C CNN
+F 0 "R5" V 5380 3250 50  0000 C CNN
 F 1 "3k3" V 5300 3250 50  0000 C CNN
 F 2 "Resistors_SMD:R_0805" H 5300 3250 60  0001 C CNN
@@
 $EndComp
 $Comp
-L R-RESCUE-emulator R6_v3
+L R-RESCUE-emulator R6
 U 1 1 52D02ABB
 P 5300 3650
-F 0 "R6_v3" V 5380 3650 50  0000 C CNN
+F 0 "R6" V 5380 3650 50  0000 C CNN
 F 1 "3k3" V 5300 3650 50  0000 C CNN
 F 2 "Resistors_SMD:R_0805" H 5300 3650 60  0001 C CNN
@@
 $EndComp
 $Comp
-L CONN_01X04 ICSP_UART_v3
+L CONN_01X04 ICSP_UART1
 U 1 1 542D83A2
 P 2650 3600
-F 0 "ICSP_UART_v3" H 2650 3900 50  0000 C CNN
+F 0 "ICSP_UART1" H 2700 3900 50  0000 C CNN
 F 1 "CONN_01X04" V 2750 3600 50  0000 C CNN
 F 2 "Pin_Headers:Pin_Header_Straight_1x04" H 2650 3600 60  0001 C CNN
@@
 	1    0    0    -1
 $EndComp
-Text Label 3150 3950 0    60   ~ 0
-MCLR_VPP
 Wire Wire Line
 	5050 5350 5050 5150
@@
 	3400 3450 2850 3450
 Wire Wire Line
-	2850 3550 3400 3550
-Wire Wire Line
 	3400 3550 3400 3650
 Wire Wire Line
@@
 	3150 4400 3150 4300
 Connection ~ 3150 3950
-$Comp
-L R-RESCUE-emulator R5_v2
-U 1 1 55C4BA7B
-P 5300 4400
-F 0 "R5_v2" V 5380 4400 50  0000 C CNN
-F 1 "3k3" V 5300 4400 50  0000 C CNN
-F 2 "Resistors_SMD:R_0805" H 5300 4400 60  0001 C CNN
-F 3 "" H 5300 4400 60  0001 C CNN
-	1    5300 4400
-	0    -1   -1   0
-$EndComp
-$Comp
-L R-RESCUE-emulator R6_v2
-U 1 1 55C4BADB
-P 5300 4700
-F 0 "R6_v2" V 5380 4700 50  0000 C CNN
-F 1 "3k3" V 5300 4700 50  0000 C CNN
-F 2 "Resistors_SMD:R_0805" H 5300 4700 60  0001 C CNN
-F 3 "" H 5300 4700 60  0001 C CNN
-	1    5300 4700
-	0    -1   -1   0
-$EndComp
 Wire Wire Line
-	5550 4400 5600 4400
-Wire Wire Line
-	5600 4400 5600 3250
-Connection ~ 5600 3250
-Wire Wire Line
-	5550 4700 5650 4700
-Wire Wire Line
-	5650 4700 5650 3650
-Connection ~ 5650 3650
-Wire Wire Line
-	2900 4400 5050 4400
-Wire Wire Line
-	5050 4700 3000 4700
-Wire Wire Line
-	3000 4700 3000 3550
-Connection ~ 3000 3550
-Wire Wire Line
-	2900 3450 2900 4400
-Connection ~ 2900 3450
-$Comp
-L CONN_01X02 UART_v2
-U 1 1 55C4D672
-P 5350 2800
-F 0 "UART_v2" H 5350 3100 50  0000 C CNN
-F 1 "CONN_01X04" V 5450 2800 50  0000 C CNN
-F 2 "Pin_Headers:Pin_Header_Straight_1x02" H 5350 2800 60  0001 C CNN
-F 3 "" H 5350 2800 60  0000 C CNN
-	1    5350 2800
-	1    0    0    -1
-$EndComp
-Wire Wire Line
-	5150 2750 4950 2750
-Wire Wire Line
-	4950 2750 4950 3250
-Connection ~ 4950 3250
-Wire Wire Line
-	5000 3650 5000 2850
-Wire Wire Line
-	5000 2850 5150 2850
-Connection ~ 5000 3650
+	2850 3550 3400 3550
 $EndSCHEMATC

Commit message: cleanup
Parts:
- renumbered C10 to C3
Connections:
- net ARCHOS: now reaches ICSP_UART1.4 (P4), U1.2 (GP5/OSC1)
- net PJRC: now reaches ICSP_UART1.3 (P3), U1.3 (GP4/OSC2)
- net RESET: now reaches C1.1, ICSP_UART1.2 (P2), R1.1, U1.4 (GP3/MCLR)
- net CLK renamed CLK-PRG_DATA
- net DataIn renamed DataIn-PRG_CLK
Other:
- moved on the sheet: ICSP_UART1
Changed lines of the file:
@@
 POWER_CTL
 $Comp
-L C-RESCUE-emulator C10
+L C-RESCUE-emulator C3
 U 1 1 52E79ABE
 P 4100 2500
-F 0 "C10" H 4150 2600 50  0000 L CNN
+F 0 "C3" H 4150 2600 50  0000 L CNN
 F 1 "100n" H 4150 2400 50  0000 L CNN
 F 2 "Capacitors_SMD:C_0805" H 4100 2500 60  0001 C CNN
@@
 $EndComp
 Text GLabel 7650 3800 0    60   Input ~ 0
-CLK
+CLK-PRG_DATA
 Text GLabel 7650 3700 0    60   Input ~ 0
-DataIn
+DataIn-PRG_CLK
 Text GLabel 7650 3600 0    60   Input ~ 0
 DataOut
@@
 DataOut
 Text GLabel 5750 3250 2    60   Input ~ 0
-CLK
+CLK-PRG_DATA
 Text GLabel 5750 3650 2    60   Input ~ 0
-DataIn
+DataIn-PRG_CLK
 $Comp
 L +5V #PWR02
@@
 L CONN_01X04 ICSP_UART1
 U 1 1 542D83A2
-P 2650 3600
-F 0 "ICSP_UART1" H 2700 3900 50  0000 C CNN
-F 1 "CONN_01X04" V 2750 3600 50  0000 C CNN
-F 2 "Pin_Headers:Pin_Header_Straight_1x04" H 2650 3600 60  0001 C CNN
-F 3 "" H 2650 3600 60  0000 C CNN
-	1    2650 3600
-	-1   0    0    1
+P 7900 4450
+F 0 "ICSP_UART1" H 7950 4750 50  0000 C CNN
+F 1 "CONN_01X04" V 8000 4450 50  0000 C CNN
+F 2 "Pin_Headers:Pin_Header_Straight_1x04" H 7900 4450 60  0001 C CNN
+F 3 "" H 7900 4450 60  0000 C CNN
+	1    7900 4450
+	1    0    0    -1
 $EndComp
 $Comp
@@
 Wire Wire Line
 	2850 3550 3400 3550
+Wire Wire Line
+	7700 4600 7600 4600
+Wire Wire Line
+	7600 4500 7700 4500
+Wire Wire Line
+	7600 4400 7700 4400
+Wire Wire Line
+	7600 4300 7700 4300
+Text GLabel 7600 4300 0    60   Input ~ 0
++5V
+Text GLabel 2850 3750 0    60   Input ~ 0
++5V
+Text GLabel 7600 4400 0    60   Input ~ 0
+RESET
+Text GLabel 2850 3650 0    60   Input ~ 0
+RESET
+Text GLabel 2850 3450 0    60   Input ~ 0
+ARCHOS
+Text GLabel 2850 3550 0    60   Input ~ 0
+PJRC
+Text GLabel 7600 4600 0    60   Input ~ 0
+ARCHOS
+Text GLabel 7600 4500 0    60   Input ~ 0
+PJRC
 $EndSCHEMATC
