File: kicad/arduino_based_cdc_emulator/atmega88_k9spud/arduino_based_cdc_emu.sch (KiCad schematic (older format))
At the start: 13 parts, among them IC1 ATMEGA88-A, P1 CONN_5, P2 CONN_2, U1 78L05, X1 20MHz

Commit message: need rework, changed kicad.....
Parts:
- added 2u2: 100n, symbol CP
- C1, C2, C3, C4: symbol C -> C-RESCUE-arduino_based_cdc_emu
- IC1: symbol ATMEGA88-A -> ATMEGA88-A-RESCUE-arduino_based_cdc_emu
- R1, R2, R3, R4: symbol R -> R-RESCUE-arduino_based_cdc_emu
Connections:
- wire segments 42 -> 45
- no-connect marks 0 -> 17
Changed lines of the file:
@@
 EESchema Schematic File Version 2
+LIBS:arduino_based_cdc_emu-rescue
 LIBS:power
 LIBS:device
@@
 LIBS:memory
 LIBS:xilinx
-LIBS:special
 LIBS:microcontrollers
 LIBS:dsp
@@
 	4250 5550 3750 5550
 Connection ~ 3850 5550
-Wire Wire Line
-	3350 5700 3350 4950
 Connection ~ 3350 5550
 Wire Wire Line
@@
 	7300 4150 6850 4150
 Wire Wire Line
-	7300 5300 6850 5300
+	6850 5300 7500 5300
 Wire Wire Line
 	6350 5300 6150 5300
@@
 $EndComp
 $Comp
-L R R3
+L R-RESCUE-arduino_based_cdc_emu R3
 U 1 1 532072FD
 P 6600 5300
@@
 DataOut
 $Comp
-L GND #PWR02
-U 1 1 530C945D
-P 9600 3400
-F 0 "#PWR02" H 9600 3400 30  0001 C CNN
-F 1 "GND" H 9600 3330 30  0001 C CNN
-F 2 "" H 9600 3400 60  0001 C CNN
-F 3 "" H 9600 3400 60  0001 C CNN
-	1    9600 3400
-	1    0    0    -1
-$EndComp
-$Comp
 L CONN_5 P1
 U 1 1 530C9435
@@
 $EndComp
 $Comp
-L +12V #PWR03
+L +12V #PWR02
 U 1 1 530C8041
 P 8550 5300
-F 0 "#PWR03" H 8550 5250 20  0001 C CNN
+F 0 "#PWR02" H 8550 5250 20  0001 C CNN
 F 1 "+12V" H 8550 5400 30  0000 C CNN
 F 2 "" H 8550 5300 60  0001 C CNN
@@
 $EndComp
 $Comp
-L +5V #PWR04
+L +5V #PWR03
 U 1 1 530C8014
 P 10000 5350
-F 0 "#PWR04" H 10000 5440 20  0001 C CNN
+F 0 "#PWR03" H 10000 5440 20  0001 C CNN
 F 1 "+5V" H 10000 5440 30  0000 C CNN
 F 2 "" H 10000 5350 60  0001 C CNN
 F 3 "" H 10000 5350 60  0001 C CNN
 	1    10000 5350
-	1    0    0    -1
-$EndComp
-$Comp
-L GND #PWR05
-U 1 1 530C800A
-P 9350 6050
-F 0 "#PWR05" H 9350 6050 30  0001 C CNN
-F 1 "GND" H 9350 5980 30  0001 C CNN
-F 2 "" H 9350 6050 60  0001 C CNN
-F 3 "" H 9350 6050 60  0001 C CNN
-	1    9350 6050
 	1    0    0    -1
 $EndComp
@@
 $EndComp
 $Comp
-L GND #PWR06
-U 1 1 530C7FEB
-P 10000 6050
-F 0 "#PWR06" H 10000 6050 30  0001 C CNN
-F 1 "GND" H 10000 5980 30  0001 C CNN
-F 2 "" H 10000 6050 60  0001 C CNN
-F 3 "" H 10000 6050 60  0001 C CNN
-	1    10000 6050
-	1    0    0    -1
-$EndComp
-$Comp
-L GND #PWR07
-U 1 1 530C7FE7
-P 8650 6050
-F 0 "#PWR07" H 8650 6050 30  0001 C CNN
-F 1 "GND" H 8650 5980 30  0001 C CNN
-F 2 "" H 8650 6050 60  0001 C CNN
-F 3 "" H 8650 6050 60  0001 C CNN
-	1    8650 6050
-	1    0    0    -1
-$EndComp
-$Comp
-L C C4
+L C-RESCUE-arduino_based_cdc_emu C4
 U 1 1 530C7FE2
 P 10000 5650
@@
 $EndComp
 $Comp
-L C C3
+L C-RESCUE-arduino_based_cdc_emu C3
 U 1 1 530C7FD9
 P 8650 5650
@@
 $EndComp
 $Comp
-L R R2
+L R-RESCUE-arduino_based_cdc_emu R2
 U 1 1 530C78F0
 P 6600 4350
@@
 $EndComp
 $Comp
-L R R1
+L R-RESCUE-arduino_based_cdc_emu R1
 U 1 1 530C77F4
 P 6600 4150
@@
 $EndComp
 $Comp
-L R R4
+L R-RESCUE-arduino_based_cdc_emu R4
 U 1 1 530C77E3
 P 6600 5650
@@
 $EndComp
 $Comp
-L +5V #PWR08
+L +5V #PWR04
 U 1 1 530C77C0
 P 4200 3650
-F 0 "#PWR08" H 4200 3740 20  0001 C CNN
+F 0 "#PWR04" H 4200 3740 20  0001 C CNN
 F 1 "+5V" H 4200 3740 30  0000 C CNN
 F 2 "" H 4200 3650 60  0001 C CNN
@@
 $EndComp
 $Comp
-L GND #PWR09
-U 1 1 530C77A6
-P 4200 6300
-F 0 "#PWR09" H 4200 6300 30  0001 C CNN
-F 1 "GND" H 4200 6230 30  0001 C CNN
-F 2 "" H 4200 6300 60  0001 C CNN
-F 3 "" H 4200 6300 60  0001 C CNN
-	1    4200 6300
-	1    0    0    -1
-$EndComp
-$Comp
-L GND #PWR010
-U 1 1 530C7791
-P 3350 5700
-F 0 "#PWR010" H 3350 5700 30  0001 C CNN
-F 1 "GND" H 3350 5630 30  0001 C CNN
-F 2 "" H 3350 5700 60  0001 C CNN
-F 3 "" H 3350 5700 60  0001 C CNN
-	1    3350 5700
-	1    0    0    -1
-$EndComp
-$Comp
-L C C2
+L C-RESCUE-arduino_based_cdc_emu C2
 U 1 1 530C7707
 P 3550 5550
@@
 $EndComp
 $Comp
-L C C1
+L C-RESCUE-arduino_based_cdc_emu C1
 U 1 1 530C7703
 P 3550 4950
@@
 $EndComp
 $Comp
-L ATMEGA88-A IC1
+L ATMEGA88-A-RESCUE-arduino_based_cdc_emu IC1
 U 1 1 530C76C5
 P 5150 4950
@@
 $EndComp
 $Comp
-L +12V #PWR011
+L +12V #PWR05
 U 1 1 543549B8
-P 9050 3250
-F 0 "#PWR011" H 9050 3200 20  0001 C CNN
-F 1 "+12V" H 9050 3350 30  0000 C CNN
-F 2 "" H 9050 3250 60  0001 C CNN
-F 3 "" H 9050 3250 60  0001 C CNN
-	1    9050 3250
-	1    0    0    -1
-$EndComp
-Wire Wire Line
-	4250 4450 4200 4450
+P 9050 3200
+F 0 "#PWR05" H 9050 3150 20  0001 C CNN
+F 1 "+12V" H 9050 3300 30  0000 C CNN
+F 2 "" H 9050 3200 60  0001 C CNN
+F 3 "" H 9050 3200 60  0001 C CNN
+	1    9050 3200
+	1    0    0    -1
+$EndComp
 Wire Wire Line
 	4200 4450 4200 3650
@@
 Wire Wire Line
 	9600 4400 9750 4400
+Wire Wire Line
+	9550 4600 9550 4500
+Wire Wire Line
+	9550 4500 9750 4500
+NoConn ~ 6150 5750
+NoConn ~ 6150 5850
+NoConn ~ 6150 5950
+NoConn ~ 6150 6050
+NoConn ~ 6150 6150
+NoConn ~ 6150 5200
+NoConn ~ 6150 5100
+NoConn ~ 6150 5000
+NoConn ~ 6150 4900
+NoConn ~ 6150 4800
+NoConn ~ 6150 4700
+NoConn ~ 6150 4550
+NoConn ~ 6150 4450
+NoConn ~ 6150 4250
+NoConn ~ 6150 4050
+NoConn ~ 6150 3950
+NoConn ~ 6150 3850
+$Comp
+L GND #PWR06
+U 1 1 564E2443
+P 4200 6300
+F 0 "#PWR06" H 4200 6050 50  0001 C CNN
+F 1 "GND" H 4200 6150 50  0000 C CNN
+F 2 "" H 4200 6300 60  0000 C CNN
+F 3 "" H 4200 6300 60  0000 C CNN
+	1    4200 6300
+	1    0    0    -1
+$EndComp
+$Comp
+L GND #PWR07
+U 1 1 564E2722
+P 3350 5700
+F 0 "#PWR07" H 3350 5450 50  0001 C CNN
+F 1 "GND" H 3350 5550 50  0000 C CNN
+F 2 "" H 3350 5700 60  0000 C CNN
+F 3 "" H 3350 5700 60  0000 C CNN
+	1    3350 5700
+	1    0    0    -1
+$EndComp
+$Comp
+L GND #PWR08
+U 1 1 564E291B
+P 8650 6050
+F 0 "#PWR08" H 8650 5800 50  0001 C CNN
+F 1 "GND" H 8650 5900 50  0000 C CNN
+F 2 "" H 8650 6050 60  0000 C CNN
+F 3 "" H 8650 6050 60  0000 C CNN
+	1    8650 6050
+	1    0    0    -1
+$EndComp
+$Comp
+L GND #PWR09
+U 1 1 564E2BE7
+P 9350 6050
+F 0 "#PWR09" H 9350 5800 50  0001 C CNN
+F 1 "GND" H 9350 5900 50  0000 C CNN
+F 2 "" H 9350 6050 60  0000 C CNN
+F 3 "" H 9350 6050 60  0000 C CNN
+	1    9350 6050
+	1    0    0    -1
+$EndComp
+$Comp
+L GND #PWR010
+U 1 1 564E2C19
+P 10000 6050
+F 0 "#PWR010" H 10000 5800 50  0001 C CNN
+F 1 "GND" H 10000 5900 50  0000 C CNN
+F 2 "" H 10000 6050 60  0000 C CNN
+F 3 "" H 10000 6050 60  0000 C CNN
+	1    10000 6050
+	1    0    0    -1
+$EndComp
+$Comp
+L GND #PWR011
+U 1 1 564E2EC9
+P 9550 4600
+F 0 "#PWR011" H 9550 4350 50  0001 C CNN
+F 1 "GND" H 9550 4450 50  0000 C CNN
+F 2 "" H 9550 4600 60  0000 C CNN
+F 3 "" H 9550 4600 60  0000 C CNN
+	1    9550 4600
+	1    0    0    -1
+$EndComp
 $Comp
 L GND #PWR012
-U 1 1 54358932
-P 9550 4600
-F 0 "#PWR012" H 9550 4600 30  0001 C CNN
-F 1 "GND" H 9550 4530 30  0001 C CNN
-F 2 "" H 9550 4600 60  0001 C CNN
-F 3 "" H 9550 4600 60  0001 C CNN
-	1    9550 4600
-	1    0    0    -1
-$EndComp
-Wire Wire Line
-	9550 4600 9550 4500
-Wire Wire Line
-	9550 4500 9750 4500
+U 1 1 564E3127
+P 9600 3400
+F 0 "#PWR012" H 9600 3150 50  0001 C CNN
+F 1 "GND" H 9600 3250 50  0000 C CNN
+F 2 "" H 9600 3400 60  0000 C CNN
+F 3 "" H 9600 3400 60  0000 C CNN
+	1    9600 3400
+	1    0    0    -1
+$EndComp
+$Comp
+L GND #PWR013
+U 1 1 564E32CC
+P 7500 5900
+F 0 "#PWR013" H 7500 5650 50  0001 C CNN
+F 1 "GND" H 7500 5750 50  0000 C CNN
+F 2 "" H 7500 5900 60  0000 C CNN
+F 3 "" H 7500 5900 60  0000 C CNN
+	1    7500 5900
+	1    0    0    -1
+$EndComp
+$Comp
+L CP 2u2
+U 1 1 564E32FE
+P 7500 5550
+F 0 "2u2" H 7550 5650 50  0000 L CNN
+F 1 "100n" H 7550 5450 50  0000 L CNN
+F 2 "" H 7500 5550 60  0001 C CNN
+F 3 "" H 7500 5550 60  0001 C CNN
+	1    7500 5550
+	1    0    0    -1
+$EndComp
+Wire Wire Line
+	7500 5900 7500 5700
+Wire Wire Line
+	7500 5300 7500 5400
+Connection ~ 7300 5300
+Wire Wire Line
+	9050 3200 9050 3250
+Wire Wire Line
+	4250 4450 4200 4450
+Wire Wire Line
+	3350 4950 3350 5700
 $EndSCHEMATC
