File: kicad/XS3868_breadboard_adapter/XS3868_breadboard_adapter.sch (KiCad schematic (older format))
At the start: 4 parts, among them J1 SCJ368R1NUS0B00G, P1 CONN_01X12, P2 CONN_01X12, U1 XS3860

Commit message: rename xs3860 to xs3868
Parts:
- U1: value XS3860 -> XS3868; symbol XS3860 -> XS3868
Changed lines of the file:
@@
 LIBS:contrib
 LIBS:valves
-LIBS:XS3860
 LIBS:phonejack
-LIBS:bt_breakout_adapter_xs3868-cache
+LIBS:SOYO-BT24G03
+LIBS:XS3868
+LIBS:XS3868_breadboard_adapter-cache
 EELAYER 25 0
 EELAYER END
@@
 $EndDescr
 $Comp
-L XS3860 U1
+L XS3868 U1
 U 1 1 5576DBD3
 P 5650 3750
-F 0 "U1" H 5650 4250 60  0000 C CNN
-F 1 "XS3860" H 5650 4350 60  0000 C CNN
+F 0 "U1" H 5650 4637 60  0000 C CNN
+F 1 "XS3868" H 5650 4531 60  0000 C CNN
 F 2 "my_modules:XS3868" H 5700 3750 60  0001 C CNN
 F 3 "" H 5700 3750 60  0000 C CNN
