File: kicad/MB-CM15113-btm-68D_breakout_adapter/MB-CM15113-btm-68D_breakout_adapter.sch (KiCad schematic (older format))
At the start: 4 parts, among them P1 CONN_01X16, P2 CONN_01X05, P3 CONN_01X16, U1 MB-CM15113

Commit message: udpates
Parts:
- P2: footprint jacks:PJ3020D -> jacks:3.5mm_stereo_jack_PJ320B
Changed lines of the file:
@@
 LIBS:MB-CM15113
 LIBS:audio_source-cache
-LIBS:bt_breakout_adapter_MB-CM15113-cache
+LIBS:MB-CM15113-btm-68D_breakout_adapter-cache
 EELAYER 25 0
 EELAYER END
@@
 F 0 "P2" H 6450 4350 50  0000 C CNN
 F 1 "CONN_01X05" V 6550 4150 50  0000 C CNN
-F 2 "jacks:PJ3020D" H 6450 4150 60  0001 C CNN
+F 2 "jacks:3.5mm_stereo_jack_PJ320B" H 6450 4150 60  0001 C CNN
 F 3 "" H 6450 4150 60  0000 C CNN
 	1    6450 4150

Commit message: updates
Parts:
- added D? (x2): D, LEDs.pretty:LED-1206, symbol D
- added R? (x2): 470, Resistors_SMD.pretty:R_0805_HandSoldering, symbol R
- added R? (x2): 10k, Resistors_SMD.pretty:R_0805_HandSoldering, symbol R
- added SW? (x2): SW_PUSH, Buttons_Switches_SMD:SW_SPST_FSMSM, symbol SW_PUSH
Connections:
- net at P1.6 (P6), U1.11 (1V8): now also R?.1
- net at P1.4 (P4), U1.13 (GND): now also SW?.2
- net at P1.2 (P2), U1.15 (RST): now also R?.2, SW?.1
- net at U1.18 (CSB): now also P3.2 (P2); no longer P3.15 (P15)
- net at P2.2 (P2), P3.14 (P14): now also U1.30 (L+); no longer U1.19 (MISO)
- net at U1.20 (GND): now also P3.4 (P4); no longer P3.13 (P13)
- net at P2.1 (P1), P3.12 (P12): now also U1.28 (AGND); no longer U1.21 (LED0)
- net at U1.22 (LED1): now also P3.6 (P6), D?.1 (K); no longer P3.11 (P11)
- net at U1.23 (VREG): now also P3.7 (P7), SW?.2; no longer P3.10 (P10)
- net at U1.24 (BAT_IN): now also P3.8 (P8), R?.1, R?.2, R?.2; no longer P3.9 (P9)
- net at U1.25 (5V+_CHARGER): now also P3.9 (P9); no longer P3.8 (P8)
- net at U1.26 (MIC_BIAS): now also P3.10 (P10); no longer P3.7 (P7)
- net at U1.27 (MIC+): now also P3.11 (P11); no longer P3.6 (P6)
- net at P3.5 (P5): now also U1.21 (LED0), D?.1 (K); no longer U1.28 (AGND)
- net at U1.29 (L-): now also P3.13 (P13); no longer P3.4 (P4)
- net at P3.3 (P3): now also U1.19 (MISO); no longer U1.30 (L+)
- net at U1.31 (R-): now also P3.15 (P15); no longer P3.2 (P2)
- net at P3.1 (P1): now also U1.17 (CLK); no longer U1.32 (R+)
- new net: P2.5 (P5), U1.32 (R+)
- new net: D?.2 (A), R?.1 (x2)
- new net: R?.2, SW?.1
- now unconnected: P3.16 (P16)
Other:
- moved on the sheet: P2, P3
Changed lines of the file:
@@
 L CONN_01X16 P3
 U 1 1 55EC639E
-P 6900 2900
-F 0 "P3" H 6900 3750 50  0000 C CNN
-F 1 "CONN_01X16" V 7000 2900 50  0000 C CNN
-F 2 "Pin_Headers:Pin_Header_Straight_1x16" H 6900 2900 60  0001 C CNN
-F 3 "" H 6900 2900 60  0000 C CNN
-	1    6900 2900
-	1    0    0    -1
+P 8300 2900
+F 0 "P3" H 8300 3750 50  0000 C CNN
+F 1 "CONN_01X16" V 8400 2900 50  0000 C CNN
+F 2 "Pin_Headers:Pin_Header_Straight_1x16" H 8300 2900 60  0001 C CNN
+F 3 "" H 8300 2900 60  0000 C CNN
+	1    8300 2900
+	1    0    0    1
 $EndComp
 $Comp
 L CONN_01X05 P2
 U 1 1 55EC6792
-P 6450 4150
-F 0 "P2" H 6450 4350 50  0000 C CNN
-F 1 "CONN_01X05" V 6550 4150 50  0000 C CNN
-F 2 "jacks:3.5mm_stereo_jack_PJ320B" H 6450 4150 60  0001 C CNN
-F 3 "" H 6450 4150 60  0000 C CNN
-	1    6450 4150
+P 6450 1650
+F 0 "P2" H 6450 1850 50  0000 C CNN
+F 1 "CONN_01X05" V 6550 1650 50  0000 C CNN
+F 2 "jacks:3.5mm_stereo_jack_PJ320B" H 6450 1650 60  0001 C CNN
+F 3 "" H 6450 1650 60  0000 C CNN
+	1    6450 1650
+	0    1    -1   0
+$EndComp
+$Comp
+L R R?
+U 1 1 57ECF44A
+P 6300 4300
+F 0 "R?" H 6370 4346 50  0000 L CNN
+F 1 "470" H 6370 4255 50  0000 L CNN
+F 2 "Resistors_SMD.pretty:R_0805_HandSoldering" H 6370 4209 50  0001 L CNN
+F 3 "" H 6300 4300 50  0000 C CNN
+	1    6300 4300
+	1    0    0    -1
+$EndComp
+$Comp
+L R R?
+U 1 1 57ECF4C4
+P 6600 4300
+F 0 "R?" H 6670 4346 50  0000 L CNN
+F 1 "470" H 6670 4255 50  0000 L CNN
+F 2 "Resistors_SMD.pretty:R_0805_HandSoldering" H 6670 4209 50  0001 L CNN
+F 3 "" H 6600 4300 50  0000 C CNN
+	1    6600 4300
+	1    0    0    -1
+$EndComp
+$Comp
+L D D?
+U 1 1 57ECF6CA
+P 6300 3900
+F 0 "D?" V 6254 3978 50  0000 L CNN
+F 1 "D" V 6345 3978 50  0000 L CNN
+F 2 "LEDs.pretty:LED-1206" V 6391 3978 50  0001 L CNN
+F 3 "" H 6300 3900 50  0000 C CNN
+	1    6300 3900
 	0    1    1    0
 $EndComp
+$Comp
+L D D?
+U 1 1 57ECF843
+P 6600 3900
+F 0 "D?" V 6554 3978 50  0000 L CNN
+F 1 "D" V 6645 3978 50  0000 L CNN
+F 2 "LEDs.pretty:LED-1206" V 6691 3978 50  0001 L CNN
+F 3 "" H 6600 3900 50  0000 C CNN
+	1    6600 3900
+	0    1    1    0
+$EndComp
 Wire Wire Line
 	4750 2150 4250 2150
@@
 	4250 3650 4750 3650
 Wire Wire Line
+	6200 3650 8100 3650
+Wire Wire Line
+	6200 3550 8100 3550
+Wire Wire Line
+	6200 3450 8100 3450
+Wire Wire Line
+	6200 3350 8100 3350
+Wire Wire Line
+	6200 3250 8100 3250
+Wire Wire Line
+	6200 3150 8100 3150
+Wire Wire Line
+	6200 3050 8100 3050
+Wire Wire Line
+	6200 2950 8100 2950
+Wire Wire Line
+	6200 2850 8100 2850
+Wire Wire Line
+	6200 2750 8100 2750
+Wire Wire Line
+	6200 2650 8100 2650
+Wire Wire Line
+	6200 2550 8100 2550
+Wire Wire Line
+	6200 2450 8100 2450
+Wire Wire Line
+	6200 2350 8100 2350
+Wire Wire Line
+	6200 2250 8100 2250
+Wire Wire Line
 	6200 2150 6700 2150
 Wire Wire Line
-	6700 2250 6200 2250
-Wire Wire Line
-	6200 2350 6700 2350
-Wire Wire Line
-	6700 2450 6200 2450
-Wire Wire Line
-	6200 2550 6700 2550
-Wire Wire Line
-	6700 2650 6200 2650
-Wire Wire Line
-	6200 2750 6700 2750
-Wire Wire Line
-	6700 2850 6200 2850
-Wire Wire Line
-	6200 2950 6700 2950
-Wire Wire Line
-	6700 3050 6200 3050
-Wire Wire Line
-	6200 3150 6700 3150
-Wire Wire Line
-	6200 3250 6700 3250
-Wire Wire Line
-	6200 3350 6700 3350
-Wire Wire Line
-	6700 3450 6200 3450
-Wire Wire Line
-	6200 3550 6700 3550
-Wire Wire Line
-	6200 3650 6700 3650
-Wire Wire Line
-	6650 3950 6650 3250
-Connection ~ 6650 3250
-Wire Wire Line
-	6550 3450 6550 3950
-Connection ~ 6550 3450
-Wire Wire Line
-	6250 3650 6250 3950
-Connection ~ 6250 3650
+	6650 1850 6650 2550
+Connection ~ 6650 2550
+Wire Wire Line
+	6550 2350 6550 1850
+Connection ~ 6550 2350
+Wire Wire Line
+	6250 2150 6250 1850
+Connection ~ 6250 2150
+Wire Wire Line
+	6300 3750 6300 3250
+Connection ~ 6300 3250
+Wire Wire Line
+	6600 3150 6600 3750
+Connection ~ 6600 3150
+Wire Wire Line
+	6300 4050 6300 4150
+Wire Wire Line
+	6600 4050 6600 4150
+Wire Wire Line
+	6300 4450 6300 4550
+Wire Wire Line
+	6300 4550 6600 4550
+Wire Wire Line
+	6600 4550 6600 4450
+Wire Wire Line
+	6450 4550 6450 2950
+Connection ~ 6450 2950
+Connection ~ 6450 4550
+$Comp
+L SW_PUSH SW?
+U 1 1 57ED00C6
+P 7050 4150
+F 0 "SW?" V 7096 4096 50  0000 R CNN
+F 1 "SW_PUSH" V 7005 4096 50  0000 R CNN
+F 2 "Buttons_Switches_SMD:SW_SPST_FSMSM" H 7050 4150 50  0001 C CNN
+F 3 "" H 7050 4150 50  0000 C CNN
+	1    7050 4150
+	0    -1   -1   0
+$EndComp
+Wire Wire Line
+	7050 3850 7050 3050
+Connection ~ 7050 3050
+Wire Wire Line
+	7050 4450 7050 4550
+Wire Wire Line
+	7050 4550 7300 4550
+Wire Wire Line
+	7300 4550 7300 4450
+$Comp
+L R R?
+U 1 1 57ED0215
+P 7300 4300
+F 0 "R?" H 7370 4346 50  0000 L CNN
+F 1 "10k" H 7370 4255 50  0000 L CNN
+F 2 "Resistors_SMD.pretty:R_0805_HandSoldering" H 7370 4209 50  0001 L CNN
+F 3 "" H 7300 4300 50  0000 C CNN
+	1    7300 4300
+	1    0    0    -1
+$EndComp
+Wire Wire Line
+	7300 4150 7300 2950
+Connection ~ 7300 2950
+$Comp
+L SW_PUSH SW?
+U 1 1 57ED066C
+P 4400 4150
+F 0 "SW?" V 4446 4096 50  0000 R CNN
+F 1 "SW_PUSH" V 4355 4096 50  0000 R CNN
+F 2 "Buttons_Switches_SMD:SW_SPST_FSMSM" H 4400 4150 50  0001 C CNN
+F 3 "" H 4400 4150 50  0000 C CNN
+	1    4400 4150
+	0    -1   -1   0
+$EndComp
+Wire Wire Line
+	4400 4450 4400 4550
+Wire Wire Line
+	4400 4550 4650 4550
+Wire Wire Line
+	4650 4550 4650 4450
+$Comp
+L R R?
+U 1 1 57ED0675
+P 4650 4300
+F 0 "R?" H 4720 4346 50  0000 L CNN
+F 1 "10k" H 4720 4255 50  0000 L CNN
+F 2 "Resistors_SMD.pretty:R_0805_HandSoldering" H 4720 4209 50  0001 L CNN
+F 3 "" H 4650 4300 50  0000 C CNN
+	1    4650 4300
+	1    0    0    -1
+$EndComp
+Wire Wire Line
+	4400 3850 4400 3350
+Connection ~ 4400 3350
+Wire Wire Line
+	4650 4150 4650 3150
+Connection ~ 4650 3150
+Wire Wire Line
+	4500 3550 4500 4550
+Connection ~ 4500 4550
+Connection ~ 4500 3550
 $EndSCHEMATC
