File: kicad/S3860M-S_breadboard_adapter/S3860M-S_breadboard_adapter.sch (KiCad schematic (older format))
At the start: 4 parts, among them J1 SCJ368R1NUS0B00G, P1 CONN_01X12, P2 CONN_01X12, U1 XS3868

Commit message: 0805 resistors as jumpers for selecting module
Parts:
- added D1, D2: LED, LEDs:LED-1206, symbol LED
- added R1: 10k, Resistors_SMD:R_0805_HandSoldering, symbol R
- added R2, R3: 470, Resistors_SMD:R_0805_HandSoldering, symbol R
- added SM_ONKEY1, SM_RESET1, SM_VOL+1, SM_VOL-1, XS_ONKEY1, XS_RESET1, XS_VOL+1, XS_VOL-1: 0, Resistors_SMD:R_0805, symbol R
- added SW1: 1, Buttons_Switches_SMD:SW_SPST_FSMSM, symbol SW_PUSH
- added SW2: ON/OFF, Buttons_Switches_SMD:SW_SPST_FSMSM, symbol SW_PUSH
- P2: footprint Pin_Headers:Pin_Header_Straight_1x12 -> Pin_Headers:Pin_Header_Straight_1x11; symbol CONN_01X12 -> CONN_01X11
Connections:
- net at P1.3 (P3), U1.11 (GND): now also SW1.1
- net at P1.2 (P2), U1.12 (VBAT): now also R1.2
- net at P1.1 (P1), U1.13 (1V8): now also D1.2 (A), D2.2 (A), SW2.1
- net at U1.14 (ONKEY): now also SM_ONKEY1.2; no longer P2.12 (P12)
- net at U1.15 (VOL+): now also SM_VOL+1.2, XS_RESET1.2; no longer P2.11 (P11)
- net at U1.16 (VOL-): now also SM_VOL-1.2, XS_ONKEY1.2; no longer P2.10 (P10)
- net at U1.17 (RESET): now also SM_RESET1.2, XS_VOL+1.2; no longer P2.9 (P9)
- net at U1.18 (NC): now also XS_VOL-1.2; no longer P2.8 (P8)
- net at P1.7 (P7), U1.7 (LED1): now also R2.2
- net at P1.6 (P6), U1.8 (LED2): now also R3.2
- new net: D1.1 (K), R2.1
- new net: D2.1 (K), R3.1
- new net ONKEY: P2.11 (P11), SM_ONKEY1.1, SW2.2, XS_ONKEY1.1
- new net RESET: P2.8 (P8), R1.1, SM_RESET1.1, SW1.2, XS_RESET1.1
- new net VOL+: P2.10 (P10), SM_VOL+1.1, XS_VOL+1.1
- new net VOL-: P2.9 (P9), SM_VOL-1.1, XS_VOL-1.1

Commit message: change jumper resistors to select module from 0402 to 0805, corect name for jack is PJ320B
Parts:
- J1: footprint my_modules:3.5mm_stereo_jack_PJ242 -> my_modules:3.5mm_stereo_jack_PJ320B
Changed lines of the file:
@@
 F 0 "J1" H 5650 2850 60  0000 C CNN
 F 1 "SCJ368R1NUS0B00G" H 5650 2300 60  0000 C CNN
-F 2 "my_modules:3.5mm_stereo_jack_PJ242" H 5650 2550 60  0001 C CNN
+F 2 "my_modules:3.5mm_stereo_jack_PJ320B" H 5650 2550 60  0001 C CNN
 F 3 "" H 5650 2550 60  0000 C CNN
 	1    5650 2550

Commit message: update for GND/VBUCK diffrence betwen S3860M-S and XS3868 module, using sMD jumpers  for selection betwen modules
Parts:
- removed SM_ONKEY1, SM_RESET1, SM_VOL+1, SM_VOL-1, XS_ONKEY1, XS_RESET1, XS_VOL+1, XS_VOL-1: 0, Resistors_SMD:R_0805, symbol R
- added GND1: GND, open-project:S_JUMPER_3, symbol JUMPER3
- added ONKEY1: ONKEY, open-project:S_JUMPER_3, symbol JUMPER3
- added RST1: RST, open-project:S_JUMPER_3, symbol JUMPER3
- added VBUCK1: VBUCK, open-project:S_JUMPER_3, symbol JUMPER3
- added VOL+1: VOL+, open-project:S_JUMPER_3, symbol JUMPER3
- added VOL-1: VOL-, open-project:S_JUMPER_3, symbol JUMPER3
- U1: value XS3868 -> S3860M-S; symbol XS3868 -> S3860M-S
- renumbered SW2 to ON/OFF/PLAY1, SW1 to RESET1
Connections:
- net ONKEY: now also ONKEY1.2
- net RESET: now also RST1.2
- net VOL+: now also VOL+1.2
- net VOL-: now also VOL-1.2
- net at U1.10 (VBUCK): now also GND1.3, VBUCK1.1; no longer P1.4 (P4)
- net GND: now reaches P1.3 (P3), RESET1.1
- net GND: now also GND1.2; no longer U1.11 (GND)
- net at U1.14 (ONKEY): now also ONKEY1.3
- net at U1.15 (VOL+): now also RST1.1, VOL+1.3
- net at U1.16 (VOL-): now also ONKEY1.1, VOL-1.3
- net at U1.17 (RESET): now also RST1.3, VOL+1.1
- net at U1.18 (NC): now also VOL-1.1
- new net: GND1.1, U1.11 (GND), VBUCK1.3
- new net VBUCK: P1.4 (P4), VBUCK1.2
Other:
- note added: "S3860M-S"
- note added: "X3860M-S"
- note added: "XS3868"
- moved on the sheet: P1

Commit message: updates, I do not remember what I changed ....
Parts:
- J1: footprint my_modules:3.5mm_stereo_jack_PJ320B -> jacks:3.5mm_stereo_jack_PJ320B
Changed lines of the file:
@@
 F 0 "J1" H 5650 2850 60  0000 C CNN
 F 1 "SCJ368R1NUS0B00G" H 5650 2300 60  0001 C CNN
-F 2 "my_modules:3.5mm_stereo_jack_PJ320B" H 5650 2550 60  0001 C CNN
+F 2 "jacks:3.5mm_stereo_jack_PJ320B" H 5650 2550 60  0001 C CNN
 F 3 "" H 5650 2550 60  0000 C CNN
 	1    5650 2550
