File: kicad/F-3188_CSR8645_breadbord_Adapter/F-3188_CSR8645_breadbord_Adapter.sch (KiCad schematic (older format))
At the start: 4 parts, among them J1 SCJ368R1NUS0B00G, P1 CONN_01X22, P2 CONN_01X21, U1 F-3188_CSR8645

Commit message: updates
Connections:
- net GND: now reaches P1.17 (P17), U1.17 (GND)
- net at P2.4 (P4), U1.40 (SPK_R_P1): now also J1.2; no longer J1.5
- net at P2.3 (P3), U1.41 (SPK_L_N1): now also J1.1
- net at P2.2 (P2), U1.42 (SPK_L_P1): now also J1.5; no longer J1.2
- net at P2.1 (P1), U1.43 (AGND): no longer J1.1
Changed lines of the file:
@@
 	6800 2700 7200 2700
-Wire Wire Line
-	7200 2800 6800 2800
 Wire Wire Line
 	6800 2900 7200 2900
@@
 Wire Wire Line
 	6000 4600 6000 4450
+Text Label 4450 4200 0    60   ~ 0
+GND
 Wire Wire Line
-	6800 2600 6800 1700
+	6850 2800 6850 1950
 Wire Wire Line
-	6900 2700 6900 1700
-Connection ~ 6900 2700
+	6850 1950 6800 1950
 Wire Wire Line
-	7150 2900 7150 1850
+	6800 1950 6800 1700
+Connection ~ 6850 2800
 Wire Wire Line
-	7150 1850 7200 1850
+	7200 2800 6800 2800
 Wire Wire Line
-	7200 1850 7200 1700
-Connection ~ 7150 2900
+	6900 1700 6900 1850
+Wire Wire Line
+	6900 1850 6950 1850
+Wire Wire Line
+	7200 1700 7200 1850
+Wire Wire Line
+	7200 1850 7150 1850
+Wire Wire Line
+	7150 1850 7150 2700
+Connection ~ 7150 2700
+Wire Wire Line
+	6950 1850 6950 2900
+Connection ~ 6950 2900
 $EndSCHEMATC
