File: kicad/audio_source/audio_source_2.kicad_pcb (KiCad board)
At the start: 2 copper layers, 20.9 x 38.8 mm, 5 parts, among them J1 SCJ368R1NUS0B00G, P1 IN, P2 OUT

Commit message: updates
Parts:
- J1: footprint jacks:SCJ-0354-5PU_no_screew -> jacks:3.5mm_stereo_jack_PJ306M_no_screw_terminal
- moved J1 4.67 mm to (112.3, 106.0)
- turned P2 to 0 degrees
Routing:
- net AGND: track 0.86 -> 71.0 mm, vias 0 -> 1
- net RADIO_left_out: track 27.5 -> 14.5 mm, vias 0 -> 1
- net CD_left_in: track 8.09 -> 11.0 mm
- net CD_right_in: track 12.1 -> 10.9 mm
- net RADIO_right_out: track 9.01 -> 9.96 mm
- net (no net): track 0.00 -> 0.61 mm
- added copper zone on F.Cu, net AGND
Other:
- board size 20.9 x 38.8 mm -> 22.9 x 37.6 mm
